Commit message: attentionpointnet

File: liche/urdf/liche.urdf (robot description, URDF)
Before this commit: robot liche, 5 links, 4 joints
Links:
- link arm: mass 947.29 -> 947.291687211666
- link base: mass 3402.9 -> 3402.94889191066
- link bucket: mass 273.21 -> 273.208189481848
Joints:
- joint arm_bucket: limit lower=-0.7 upper=1 effort=0 velocity=1 -> lower=-2.4086 upper=0.54105 effort=0 velocity=1; origin xyz=-0.27546 -1.4745 0 rpy=0 0 0 -> xyz=-0.001224 -1.5 0 rpy=0 0 0
- joint base_body: limit lower=-3 upper=3 effort=0 velocity=1 -> lower=-3.14 upper=3.14 effort=0 velocity=1; origin xyz=0.48559 0.87696 0.60176 rpy=0 -0.0023651 -1.5708 -> xyz=0 0 0.78635 rpy=0 0 0
- joint body_boom: axis 0 0 -1 -> 0 0 1; limit lower=-0.45 upper=1 effort=0 velocity=1 -> lower=-0.3 upper=1.0297 effort=0 velocity=1; origin xyz=0.27302 -0.0033226 0.1846 rpy=1.5708 0 0 -> xyz=0.27302 -0.0033226 0 rpy=1.5708 0 0
- joint boom_arm: limit lower=-0.45 upper=1 effort=0 velocity=1 -> lower=-0.87266 upper=0.59813 effort=0 velocity=1; origin xyz=2.6634 1.6057 0 rpy=0 0 -0.0023651 -> xyz=3.11 -0.0036336 0 rpy=0 0 -0.0023651
